Commit message: Skid drive plugin

File: models/urdf/ugv_description.xacro (robot description, xacro)
@@ -128,5 +128,5 @@
   <parent link="link1_1"/>
   <child link="link2_1"/>
-  <axis xyz="0.0 -0.999905 -0.013764"/>
+  <axis xyz="0.0 1.0 0.0"/>
 </joint>
 <joint name="FR Motor" type="continuous">
@@ -134,5 +134,5 @@
   <parent link="link1_1"/>
   <child link="link3_1"/>
-  <axis xyz="0.0 0.999905 0.013764"/>
+  <axis xyz="0.0 1.0 0.0"/>
 </joint>
 <joint name="RR Motor" type="continuous">
@@ -146,5 +146,5 @@
   <parent link="base_link"/>
   <child link="link4_1"/>
-  <axis xyz="0.0 -1.0 -0.0"/>
+  <axis xyz="0.0 1.0 0.0"/>
 </joint>
 <joint name="Pivot" type="revolute">

Commit message: laser plugin

File: models/urdf/ugv_description.xacro (robot description, xacro)
@@ -124,4 +124,10 @@
   </collision>
 </link>
+<link name="lidar_link"/>
+<joint name="lidar_joint" type="fixed">
+  <origin xyz="0 0 0.5" rpy="0 0 0"/>
+  <parent link="base_link"/>
+  <child link="lidar_link"/>
+</joint>
 <joint name="FL Motor" type="continuous">
   <origin xyz="-0.03 -0.27996 -0.004853" rpy="0 0 0"/>
